File: pcb/io.kicad_pcb (KiCad board)
At the start: 2 copper layers, 36.2 x 38.1 mm, 73 parts, among them Q1 AO3400A, Q10 AO3400A, Q11 AO3400A, Q12 AO3400A, Q13 AO3400A, Q14 AO3400A, Q15 AO3400A, Q16 AO3400A, Q2 AO3400A, Q3 AO3400A, Q4 AO3400A, Q5 AO3400A, Q6 AO3400A, Q7 AO3400A, Q8 AO3400A, Q9 AO3400A

Commit message: Hmmmm
Parts:
- removed D10, D11, D12, D13, D14, D15, D16, D9: LED, LED_SMD:LED_0603_1608Metric
- removed Q10, Q11, Q12, Q13, Q14, Q15, Q16, Q9: AO3400A, Package_TO_SOT_SMD:SOT-23
- removed the R17 at (149.4, 135.3)
- removed the R18 at (148.6, 139.7)
- removed the R20 at (114.9, 147.9)
- removed the R21 at (115.7, 154.3)
- removed the R23 at (149.4, 146.1)
- removed the R24 at (148.6, 150.5)
- removed R25, R27, R29, R31: 10k, Resistor_SMD:R_0603_1608Metric
- removed R26, R28, R30, R32: 440, Resistor_SMD:R_0603_1608Metric
- removed SW0: ~, iolib:TS-1088R-02526
- added C1: 100nF, Capacitor_SMD:C_0603_1608Metric, F.Cu at (136.5, 82.5)
- added C2: 100nF, Capacitor_SMD:C_0603_1608Metric, F.Cu at (141.6, 82.5)
- added C3: 100nF, Capacitor_SMD:C_0603_1608Metric, F.Cu at (146.7, 82.5)
- added C4: 100nF, Capacitor_SMD:C_0603_1608Metric, F.Cu at (151.8, 82.5)
- added C5: 100nF, Capacitor_SMD:C_0603_1608Metric, F.Cu at (156.8, 82.5)
- added C6: 100nF, Capacitor_SMD:C_0603_1608Metric, F.Cu at (161.9, 82.5)
- added C7: 100nF, Capacitor_SMD:C_0603_1608Metric, F.Cu at (167.0, 82.5)
- added C8: 100nF, Capacitor_SMD:C_0603_1608Metric, F.Cu at (172.1, 82.5)
- added R1: 220, Resistor_SMD:R_0603_1608Metric, F.Cu at (136.5, 84.5)
- added R10: 220, Resistor_SMD:R_0603_1608Metric, F.Cu at (151.8, 84.5)
- added R13: 220, Resistor_SMD:R_0603_1608Metric, F.Cu at (156.8, 84.5)
- added R16: 220, Resistor_SMD:R_0603_1608Metric, F.Cu at (161.9, 84.5)
- added R4: 220, Resistor_SMD:R_0603_1608Metric, F.Cu at (141.6, 84.5)
- added R7: 220, Resistor_SMD:R_0603_1608Metric, F.Cu at (146.7, 84.5)
- added SW8: ~, iolib:TS-1088R-02526, F.Cu at (172.1, 76.2)
- J1: footprint Connector_PinHeader_2.54mm:PinHeader_2x15_P2.54mm_Horizontal -> Connector_PinHeader_2.54mm:PinHeader_2x06_P2.54mm_Horizontal
- R19: value 10k -> 220
- R22: value 440 -> 220
- moved R22 93.7 mm to (172.1, 84.5)
- moved R8 87.8 mm to (146.7, 80.6)
- moved Q3 86.0 mm to (146.7, 87.0)
- moved R23 85.9 mm to (172.1, 80.6)
- moved D3 85.5 mm to (146.7, 91.4)
- moved R9 84.6 mm to (146.7, 89.5)
- moved Q8 83.4 mm to (172.1, 87.0)
- moved D8 82.8 mm to (172.1, 91.4)
- moved R24 82.4 mm to (172.1, 89.5)
- moved R19 78.2 mm to (167.0, 84.5)
- moved R14 69.8 mm to (156.8, 80.6)
- moved Q5 66.6 mm to (156.8, 87.0)
- moved R15 66.0 mm to (156.8, 89.5)
- moved D5 65.9 mm to (156.8, 91.4)
- moved R20 64.6 mm to (167.0, 80.6)
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- renumbered R7 to R11, R8 to R12, R9 to R14, R10 to R15, R11 to R17, R12 to R18, R1 to R2, R13 to R20, R14 to R21, R15 to R23, R16 to R24, R2 to R3, R3 to R5, R4 to R6, R5 to R8, R6 to R9
Connections:
- J1 pad 1: unconnected-(J1-Pad1) -> +3.3V
- J1 pad 10: unconnected-(J1-Pad10) -> L0_2
- J1 pad 11: unconnected-(J1-Pad11) -> L0_1
- J1 pad 12: unconnected-(J1-Pad12) -> L0_0
- J1 pad 2: unconnected-(J1-Pad2) -> +3.3V
- J1 pad 3: unconnected-(J1-Pad3) -> GND
- J1 pad 4: unconnected-(J1-Pad4) -> GND
- J1 pad 5: unconnected-(J1-Pad5) -> L0_7
- J1 pad 6: unconnected-(J1-Pad6) -> L0_6
- J1 pad 7: unconnected-(J1-Pad7) -> L0_5
- J1 pad 8: unconnected-(J1-Pad8) -> L0_4
- J1 pad 9: unconnected-(J1-Pad9) -> L0_3
- Q1 pad 1: L0_0 -> Net-(Q1-Pad1)
- Q2 pad 1: L0_1 -> Net-(Q2-Pad1)
- Q3 pad 1: L0_2 -> Net-(Q3-Pad1)
- Q4 pad 1: L0_3 -> Net-(Q4-Pad1)
- Q5 pad 1: L0_4 -> Net-(Q5-Pad1)
- Q6 pad 1: L0_5 -> Net-(Q6-Pad1)
- Q7 pad 1: L0_6 -> Net-(Q7-Pad1)
- Q8 pad 1: L0_7 -> Net-(Q8-Pad1)
- R11 pad 1: L0_3 -> Net-(Q4-Pad1)
- R14 pad 1: L0_4 -> Net-(Q5-Pad1)
- R17 pad 1: L0_5 -> Net-(Q6-Pad1)
- R19 pad 1: L1_1 -> Net-(Q7-Pad1)
- R19 pad 2: GND -> L0_6
- R2 pad 1: L0_0 -> Net-(Q1-Pad1)
- R20 pad 1: L0_6 -> Net-(Q7-Pad1)
- R22 pad 1: Net-(D11-Pad1) -> Net-(Q8-Pad1)
- R22 pad 2: Net-(Q11-Pad3) -> L0_7
- R23 pad 1: L0_7 -> Net-(Q8-Pad1)
- R5 pad 1: L0_1 -> Net-(Q2-Pad1)
- R8 pad 1: L0_2 -> Net-(Q3-Pad1)
- SW1 pad 1: L1_1 -> Net-(Q1-Pad1)
- SW2 pad 1: L1_2 -> Net-(Q2-Pad1)
- SW3 pad 1: L1_3 -> Net-(Q3-Pad1)
- SW4 pad 1: L1_4 -> Net-(Q4-Pad1)
- SW5 pad 1: L1_5 -> Net-(Q5-Pad1)
- SW6 pad 1: L1_6 -> Net-(Q6-Pad1)
- SW7 pad 1: L1_7 -> Net-(Q7-Pad1)
Routing:
- net +3.3V: track 0.00 -> 104.5 mm
- net L0_0: track 0.00 -> 47.1 mm, vias 0 -> 1
- net L0_1: track 0.00 -> 39.0 mm, vias 0 -> 1
- net L0_2: track 0.00 -> 35.3 mm, vias 0 -> 1
- net L0_3: track 0.00 -> 27.3 mm, vias 0 -> 1
- net L0_4: track 0.00 -> 25.5 mm, vias 0 -> 1
- net L0_5: track 0.00 -> 17.6 mm, vias 0 -> 1
- net L0_6: track 0.00 -> 15.6 mm, vias 0 -> 1
- net Net-(Q4-Pad1): track 0.00 -> 8.05 mm
- net Net-(Q2-Pad1): track 0.00 -> 8.05 mm
- net Net-(Q8-Pad1): track 0.00 -> 8.05 mm
- net Net-(Q6-Pad1): track 0.00 -> 8.05 mm
- net Net-(Q1-Pad1): track 0.00 -> 8.05 mm
- net Net-(Q7-Pad1): track 0.00 -> 8.05 mm
- net Net-(Q5-Pad1): track 0.00 -> 8.05 mm
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- added copper zone on B.Cu, net GND
- added copper zone on F.Cu, net GND
Other:
- board size 36.2 x 38.1 mm -> 48.9 x 21 mm
- board text added: "${TITLE} rev. ${REVISION} (C) 2022 ${AUTHOR}"
- board text added: "JLCJLCJLCJLC"
