File: pcb/io.kicad_pcb (KiCad board)
At the start: 2 copper layers, 48.9 x 21 mm, 57 parts, among them Q1 AO3400A, Q2 AO3400A, Q3 AO3400A, Q4 AO3400A, Q5 AO3400A, Q6 AO3400A, Q7 AO3400A, Q8 AO3400A

Commit message: Bumped revision
Routing:
- net L0_1: track 39.0 -> 37.9 mm
- net L0_4: track 25.5 -> 26.5 mm
Changed lines of the file:
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@@
   (segment (start 142.43 84.455) (end 143.51 84.455) (width 0.2286) (layer "F.Cu") (net 18))
   (via (at 143.51 84.455) (size 0.7) (drill 0.35) (layers "F.Cu" "B.Cu") (net 18))
-  (segment (start 178.5 88.9) (end 177.23 90.17) (width 0.2286) (layer "B.Cu") (net 18))
-  (segment (start 149.225 90.17) (end 143.51 84.455) (width 0.2286) (layer "B.Cu") (net 18))
-  (segment (start 177.23 90.17) (end 149.225 90.17) (width 0.2286) (layer "B.Cu") (net 18))
+  (segment (start 178.5 88.9) (end 147.955 88.9) (width 0.2286) (layer "B.Cu") (net 18))
+  (segment (start 147.955 88.9) (end 143.51 84.455) (width 0.2286) (layer "B.Cu") (net 18))
   (segment (start 147.51 84.455) (end 148.59 84.455) (width 0.2286) (layer "F.Cu") (net 19))
   (via (at 148.59 84.455) (size 0.7) (drill 0.35) (layers "F.Cu" "B.Cu") (net 19))
@@
   (segment (start 157.67 84.455) (end 158.75 84.455) (width 0.2286) (layer "F.Cu") (net 23))
   (via (at 158.75 84.455) (size 0.7) (drill 0.35) (layers "F.Cu" "B.Cu") (net 23))
-  (segment (start 179.6167 85.2433) (end 181.04 83.82) (width 0.2286) (layer "B.Cu") (net 23))
-  (segment (start 158.75 84.455) (end 161.035501 86.740501) (width 0.2286) (layer "B.Cu") (net 23))
-  (segment (start 176.117609 86.740501) (end 177.61481 85.2433) (width 0.2286) (layer "B.Cu") (net 23))
-  (segment (start 177.61481 85.2433) (end 179.6167 85.2433) (width 0.2286) (layer "B.Cu") (net 23))
-  (segment (start 161.035501 86.740501) (end 176.117609 86.740501) (width 0.2286) (layer "B.Cu") (net 23))
+  (segment (start 179.9233 82.7033) (end 177.6967 82.7033) (width 0.2286) (layer "B.Cu") (net 23))
+  (segment (start 174.85 85.55) (end 166.65 85.55) (width 0.2286) (layer "B.Cu") (net 23))
+  (segment (start 166.65 85.55) (end 164.3 83.2) (width 0.2286) (layer "B.Cu") (net 23))
+  (segment (start 181.04 83.82) (end 179.9233 82.7033) (width 0.2286) (layer "B.Cu") (net 23))
+  (segment (start 177.6967 82.7033) (end 174.85 85.55) (width 0.2286) (layer "B.Cu") (net 23))
+  (segment (start 164.3 83.2) (end 160.005 83.2) (width 0.2286) (layer "B.Cu") (net 23))
+  (segment (start 160.005 83.2) (end 158.75 84.455) (width 0.2286) (layer "B.Cu") (net 23))
   (segment (start 157.7825 89.4225) (end 157.67 89.535) (width 0.2286) (layer "F.Cu") (net 24))
   (segment (start 157.7825 86.995) (end 157.7825 89.4225) (width 0.2286) (layer "F.Cu") (net 24))
   (segment (start 162.75 84.455) (end 163.83 84.455) (width 0.2286) (layer "F.Cu") (net 25))
   (via (at 163.83 84.455) (size 0.7) (drill 0.35) (layers "F.Cu" "B.Cu") (net 25))
-  (segment (start 163.83 84.455) (end 165.735 86.36) (width 0.2286) (layer "B.Cu") (net 25))
-  (segment (start 165.735 86.36) (end 175.96 86.36) (width 0.2286) (layer "B.Cu") (net 25))
-  (segment (start 175.96 86.36) (end 178.5 83.82) (width 0.2286) (layer "B.Cu") (net 25))
+  (segment (start 165.735 86.36) (end 163.83 84.455) (width 0.2286) (layer "B.Cu") (net 25))
+  (segment (start 178.5 83.82) (end 175.96 86.36) (width 0.2286) (layer "B.Cu") (net 25))
+  (segment (start 175.96 86.36) (end 165.735 86.36) (width 0.2286) (layer "B.Cu") (net 25))
   (segment (start 162.8625 86.995) (end 162.8625 89.4225) (width 0.2286) (layer "F.Cu") (net 26))
   (segment (start 162.8625 89.4225) (end 162.75 89.535) (width 0.2286) (layer "F.Cu") (net 26))
   (segment (start 167.83 84.455) (end 168.91 84.455) (width 0.2286) (layer "F.Cu") (net 27))
   (via (at 168.91 84.455) (size 0.7) (drill 0.35) (layers "F.Cu" "B.Cu") (net 27))
-  (segment (start 170.18 85.725) (end 174.625 85.725) (width 0.2286) (layer "B.Cu") (net 27))
-  (segment (start 168.91 84.455) (end 170.18 85.725) (width 0.2286) (layer "B.Cu") (net 27))
-  (segment (start 174.625 85.725) (end 177.6467 82.7033) (width 0.2286) (layer "B.Cu") (net 27))
-  (segment (start 179.6167 82.7033) (end 181.04 81.28) (width 0.2286) (layer "B.Cu") (net 27))
-  (segment (start 177.6467 82.7033) (end 179.6167 82.7033) (width 0.2286) (layer "B.Cu") (net 27))
+  (segment (start 179.9233 80.1633) (end 173.2017 80.1633) (width 0.2286) (layer "B.Cu") (net 27))
+  (segment (start 173.2017 80.1633) (end 168.91 84.455) (width 0.2286) (layer "B.Cu") (net 27))
+  (segment (start 181.04 81.28) (end 179.9233 80.1633) (width 0.2286) (layer "B.Cu") (net 27))
   (segment (start 167.9425 89.4225) (end 167.83 89.535) (width 0.2286) (layer "F.Cu") (net 28))
   (segment (start 167.9425 86.995) (end 167.9425 89.4225) (width 0.2286) (layer "F.Cu") (net 28))
