File: pcb/LED.kicad_sch (KiCad schematic)
At the start: 7 parts, among them Q8 AO3400A

Commit message: Bumped revision
Parts:
- renumbered C1 to C8, R1 to R22
Changed lines of the file:
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@@
   (symbol (lib_id "Device:R") (at 119.38 95.25 270) (unit 1)
     (in_bom yes) (on_board yes)
-    (property "Reference" "R1" (id 0) (at 116.84 92.71 90))
+    (property "Reference" "R22" (id 0) (at 116.84 92.71 90))
     (property "Value" "220" (id 1) (at 121.92 92.71 90))
     (property "Footprint" "Resistor_SMD:R_0603_1608Metric" (id 2) (at 119.38 93.472 90)
@@
   (symbol (lib_id "Device:C") (at 128.27 101.6 0) (unit 1)
     (in_bom yes) (on_board yes)
-    (property "Reference" "C1" (id 0) (at 128.27 99.06 0)
+    (property "Reference" "C8" (id 0) (at 128.27 99.06 0)
       (effects (font (size 1.27 1.27)) (justify left))
     )
@@
   (symbol (lib_id "Device:LED") (at 146.05 73.66 90) (unit 1)
     (in_bom yes) (on_board yes)
-    (property "Reference" "D8" (id 0) (at 143.51 76.2 0))
-    (property "Value" "LED" (id 1) (at 143.51 72.39 0))
+    (property "Reference" "D8" (id 0) (at 143.51 73.66 0))
+    (property "Value" "LED" (id 1) (at 143.51 72.39 0)
+      (effects (font (size 1.27 1.27)) hide)
+    )
     (property "Footprint" "LED_SMD:LED_0603_1608Metric" (id 2) (at 146.05 73.66 0)
       (effects (font (size 1.27 1.27)) hide)
@@
   (symbol (lib_id "power:GND") (at 128.27 110.49 0) (unit 1)
     (in_bom yes) (on_board yes)
-    (property "Reference" "#PWR05" (id 0) (at 128.27 116.84 0)
+    (property "Reference" "#PWR033" (id 0) (at 128.27 116.84 0)
       (effects (font (size 1.27 1.27)) hide)
     )
