File: pcb/io.kicad_sch (KiCad schematic)
At the start: 9 parts

Commit message: Hmmmm
Parts:
- removed J1: ~, Connector_PinHeader_2.54mm:PinHeader_2x15_P2.54mm_Horizontal, symbol Connector_Generic:Conn_02x15_Odd_Even
- removed SW0, SW1, SW2, SW3, SW4, SW5, SW6, SW7: ~, iolib:TS-1088R-02526, symbol Switch:SW_Push
- added J1: ~, Connector_PinHeader_2.54mm:PinHeader_2x06_P2.54mm_Horizontal, symbol Connector_Generic:Conn_02x06_Odd_Even
Connections:
- net +3.3V: now also J1.1 (Pin_1), J1.2 (Pin_2)
- net L0_0: now also J1.12 (Pin_12)
- net L0_1: now also J1.11 (Pin_11)
- net L0_2: now also J1.10 (Pin_10)
- net L0_3: now also J1.9 (Pin_9)
- net L0_4: now also J1.8 (Pin_8)
- net L0_5: now also J1.7 (Pin_7)
- net L0_6: now also J1.6 (Pin_6)
- net L0_7: now also J1.5 (Pin_5)
- new net GND: J1.3 (Pin_3), J1.4 (Pin_4)
Other:
- removed sheet LED1_0
- removed sheet LED1_1
- removed sheet LED1_2
- removed sheet LED1_3
- removed sheet LED1_4
- removed sheet LED1_5
- removed sheet LED1_6
- removed sheet LED1_7
- sheet LED0_0 ports: added none; removed B
- sheet LED0_1 ports: added none; removed B
- sheet LED0_2 ports: added none; removed B
- sheet LED0_3 ports: added none; removed B
- sheet LED0_4 ports: added none; removed B
- sheet LED0_5 ports: added none; removed B
- sheet LED0_6 ports: added none; removed B
- sheet LED0_7 ports: added none; removed B

Commit message: Bumped revision
Other:
- title: (none) -> ${TITLE}
Changed lines of the file:
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@@
 (kicad_sch (version 20211123) (generator eeschema)
   (paper "A4")
+  (title_block
+    (title "${TITLE}")
+    (rev "${REVISION}")
+  )
   (wire (pts (xy 86.36 83.82) (xy 86.36 96.52))
     (stroke (width 0) (type default) (color 0 0 0 0))
